File: pcb/swallowtail.sch (KiCad schematic (older format))
At the start: 104 parts, among them J1 MJ-4PP-9, J2 Conn_01x04, SW1 SW_PUSH, SW10 SW_PUSH, SW11 SW_PUSH, SW12 SW_PUSH, SW13 SW_PUSH, SW14 SW_PUSH, SW15 SW_PUSH, SW16 SW_PUSH, SW17 SW_PUSH, SW18 SW_PUSH, SW19 SW_PUSH, SW2 SW_PUSH, SW20 SW_PUSH, SW21 SW_PUSH, SW22 SW_PUSH, SW23 SW_PUSH, SW24 SW_PUSH, SW25 SW_PUSH, SW26 SW_PUSH, SW27 SW_PUSH, SW28 SW_PUSH, SW29 SW_PUSH, SW3 SW_PUSH, SW30 SW_PUSH, SW4 SW_PUSH, SW5 SW_PUSH, SW6 SW_PUSH, SW7 SW_PUSH, SW8 SW_PUSH, SW9 SW_PUSH, U1 ProMicro_r

Commit message: v2 design
Parts:
- U1: footprint kbd:ProMicro_v2 -> swallowtail:ProMicro_v2_mod
Changed lines of the file:
@@
 F 0 "U1" H 2150 2637 60  0000 C CNN
 F 1 "ProMicro_r" H 2150 2531 60  0000 C CNN
-F 2 "kbd:ProMicro_v2" H 2250 600 60  0001 C CNN
+F 2 "swallowtail:ProMicro_v2_mod" H 2250 600 60  0001 C CNN
 F 3 "" H 2250 600 60  0000 C CNN
 	1    2100 1650
